Commit message: update to gz

File: xarm_description/urdf/common/common.gazebo.xacro (robot description, xacro)
@@ -8,4 +8,14 @@
         </xacro:if>
         <!-- <controller_manager_node_name>${prefix}controller_manager</controller_manager_node_name> -->
+      </plugin>
+    </gazebo>
+  </xacro:macro>
+  <!-- ros_gz plugin -->
+  <xacro:macro name="gz_ros2_control_plugin" params="prefix:='' ros2_control_params:=''">
+    <gazebo>
+      <plugin filename="gz_ros2_control-system" name="gz_ros2_control::GazeboSimROS2ControlPlugin">
+        <xacro:if value="${ros2_control_params != ''}">
+          <parameters>${ros2_control_params}</parameters>
+        </xacro:if>
       </plugin>
     </gazebo>

File: xarm_description/urdf/common/common.link.xacro (robot description, xacro)
@@ -28,5 +28,6 @@
       <geometry>
         <xacro:if value="${add_mesh_suffix}">
-          <mesh filename="${mesh_path}/${mesh_filename}.${mesh_suffix}"/>
+          <!-- <mesh filename="${mesh_path}/${mesh_filename}.${mesh_suffix}"/> -->
+          <mesh filename="$(find xarm_description)/meshes/${mesh_filename}.${mesh_suffix}"/>
         </xacro:if>
         <xacro:unless value="${add_mesh_suffix}">
@@ -47,5 +48,6 @@
       <geometry>
         <xacro:if value="${add_mesh_suffix}">
-          <mesh filename="${mesh_path}/${mesh_filename}.${mesh_suffix}"/>
+          <!-- <mesh filename="${mesh_path}/${mesh_filename}.${mesh_suffix}"/> -->
+          <mesh filename="$(find xarm_description)/meshes/${mesh_filename}.${mesh_suffix}"/>
         </xacro:if>
         <xacro:unless value="${add_mesh_suffix}">

File: xarm_description/urdf/xarm_device_macro.xacro (robot description, xacro)
@@ -52,10 +52,9 @@
     <!-- Specify Mesh file path -->
     <xacro:property name="mesh_suffix" value="${mesh_suffix}" scope="parent"/>
-    <xacro:if value="${ros2_control_plugin == 'gazebo_ros2_control/GazeboSystem' or ros2_control_plugin == 'ign_ros2_control/IgnitionSystem'}">
-      <!-- gazebo use -->
+    <xacro:if value="${ros2_control_plugin == 'gz_ros2_control/GazeboSimSystem'}">
+      <xacro:property name="mesh_path" value="package://xarm_description/meshes" scope="parent"/>
+    </xacro:if>
+    <xacro:unless value="${ros2_control_plugin == 'gz_ros2_control/GazeboSimSystem'}">
       <xacro:property name="mesh_path" value="file://$(find xarm_description)/meshes" scope="parent"/>
-    </xacro:if>
-    <xacro:unless value="${ros2_control_plugin == 'gazebo_ros2_control/GazeboSystem' or ros2_control_plugin == 'ign_ros2_control/IgnitionSystem'}">
-      <xacro:property name="mesh_path" value="package://xarm_description/meshes" scope="parent"/>
     </xacro:unless>
     <!-- include common.link.xacro -->
@@ -276,8 +275,8 @@
           <xacro:property name="new_ros2_control_params" value="${ros2_control_params}"/>
         </xacro:if>
-        <xacro:if value="${ros2_control_plugin == 'ign_ros2_control/IgnitionSystem'}">
-          <xacro:ignition_ros2_control_plugin prefix="${prefix}" ros2_control_params="${new_ros2_control_params}"/>
+        <xacro:if value="${ros2_control_plugin == 'gz_ros2_control/GazeboSimSystem'}">
+          <xacro:gz_ros2_control_plugin prefix="${prefix}" ros2_control_params="${new_ros2_control_params}"/>
         </xacro:if>
-        <xacro:unless value="${ros2_control_plugin == 'ign_ros2_control/IgnitionSystem'}">
+        <xacro:unless value="${ros2_control_plugin == 'gz_ros2_control/GazeboSimSystem'}">
           <xacro:gazebo_ros2_control_plugin ros2_control_params="${new_ros2_control_params}"/>
         </xacro:unless>
